Commit message: Update my_robot.xacro

File: src/my_robot/urdf/my_robot.xacro (robot description, xacro)
@@ -55,17 +55,49 @@
     </visual>
   </link>
-<link name='SIDE_wheel'>
-<inertial>
-<mass value ="5"/>
-<origin xyz="0 0 0" rpy=" 0 1.5707 1.5707"/>
-<inertia
-	ixx="0.1" ixy="0" ixz="0"
-	iyy="0.1" iyz="0"
-	izz="0.1"
-/>
-</inertial>
-<collision name ='left_SIDE_wheel'>
-<origin xyz="0 0 0" rpy=" 0 1.5707 1.5707"/>
-<geometry>
-<cylinder radius="0.1" length="0.05">
+<link name="left_wheel">
+    <inertial>
+      <mass value="5.0" />
+      <origin xyz="0 0 0" rpy="0 1.5707 1.5707" />
+      <inertia
+        ixx="0.1" ixy="0" ixz="0"
+        iyy="0.1" iyz="0"
+        izz="0.1"
+      />
+    </inertial>
+    <collision>
+      <origin xyz="0 0 0" rpy="0 1.5707 1.5707" />
+      <geometry>
+        <cylinder radius="0.1" length="0.05" />
+      </geometry>
+    </collision>
+    <visual>
+      <origin xyz="0 0 0" rpy="0 1.5707 1.5707" />
+      <geometry>
+        <cylinder radius="0.1" length="0.05" />
+      </geometry>
+    </visual>
+  <link name="right_wheel">
+    <inertial>
+      <mass value="5.0" />
+      <origin xyz="0 0 0" rpy="0 1.5707 1.5707" />
+      <inertia
+        ixx="0.1" ixy="0" ixz="0"
+        iyy="0.1" iyz="0"
+        izz="0.1"
+      />
+    </inertial>
+    <collision>
+      <origin xyz="0 0 0" rpy="0 1.5707 1.5707" />
+      <geometry>
+        <cylinder radius="0.1" length="0.05" />
+      </geometry>
+    </collision>
+    <visual>
+      <origin xyz="0 0 0" rpy="0 1.5707 1.5707" />
+      <geometry>
+        <cylinder radius="0.1" length="0.05" />
+      </geometry>
+    </visual>
+  </link>
+  </link>
 </robot>

Commit message: Update my_robot.xacro

File: src/my_robot/urdf/my_robot.xacro (robot description, xacro)
@@ -100,4 +100,20 @@
     </visual>
   </link>
+    <joint type="continuous" name="left_wheel_hinge">
+    <origin xyz="0 0.5 0" rpy="0 0 0" />
+    <child link="left_wheel" />
+    <parent link="chassis" />
+    <axis xyz="0 1 0" rpy="0 0 0" />
+    <limit effort="10000" velocity="1000" />
+    <dynamics damping="1.0" friction="1.0" />
+  </joint>
+  <joint type="continuous" name="right_wheel_hinge">
+    <origin xyz="0 -0.5 0" rpy="0 0 0" />
+    <child link="right_wheel" />
+    <parent link="chassis" />
+    <axis xyz="0 1 0" rpy="0 0 0" />
+    <limit effort="10000" velocity="1000" />
+    <dynamics damping="1.0" friction="1.0" />
+  </joint>
   </link>
 </robot>

Commit message: Update my_robot.xacro

File: src/my_robot/urdf/my_robot.xacro (robot description, xacro)
@@ -101,5 +101,5 @@
   </link>
     <joint type="continuous" name="left_wheel_hinge">
-    <origin xyz="0 0.5 0" rpy="0 0 0" />
+    <origin xyz="0 0.15 0" rpy="0 0 0" />
     <child link="left_wheel" />
     <parent link="chassis" />
@@ -109,5 +109,5 @@
   </joint>
   <joint type="continuous" name="right_wheel_hinge">
-    <origin xyz="0 -0.5 0" rpy="0 0 0" />
+    <origin xyz="0 -0.15 0" rpy="0 0 0" />
     <child link="right_wheel" />
     <parent link="chassis" />

Commit message: Update my_robot.xacro

File: src/my_robot/urdf/my_robot.xacro (robot description, xacro)
@@ -116,4 +116,27 @@
     <dynamics damping="1.0" friction="1.0" />
   </joint>
+  <link name= 'camera'/>
+  <pose>0 0 0 0 0 0</pose>
+   <inertial>
+      <mass value="5.0" />
+      <origin xyz="0 0 0" rpy="0 0 0" />
+      <inertia
+        ixx="1e-6" ixy="0" ixz="0"
+        iyy="1e-6" iyz="0"
+        izz="1e-6"
+      />
+    </inertial>
+    <collision name='collision_camera'>
+      <origin xyz="0 0 0" rpy=" 0 0 0"/>
+      <geometry>
+        <box size=".05 .05 .05"/>
+      </geometry>
+    </collision>
+ <visual name='camera_visual'>
+      <origin xyz="0 0 0" rpy=" 0 0 0"/>
+      <geometry>
+        <box size=".05 .05 .05"/>
+      </geometry>
+    </visual>
   </link>
 </robot>

Commit message: Update my_robot.xacro

File: src/my_robot/urdf/my_robot.xacro (robot description, xacro)
@@ -127,5 +127,5 @@
       />
     </inertial>
-    <collision name='collision_camera'>
+    <collision name='camera_collision'>
       <origin xyz="0 0 0" rpy=" 0 0 0"/>
       <geometry>

Commit message: Update my_robot.xacro

File: src/my_robot/urdf/my_robot.xacro (robot description, xacro)
@@ -139,4 +139,11 @@
       </geometry>
     </visual>
+  <joint type="fixed" name="camer_joint">
+    <origin xyz="0.2 0 0" rpy="0 0 0" />
+    <child link="left_wheel" />
+    <parent link="chassis" />
+    <axis xyz="0 1 0" rpy="0 0 0" />
+  </joint>
+  </link>
   </link>
 </robot>

Commit message: Update my_robot.xacro

File: src/my_robot/urdf/my_robot.xacro (robot description, xacro)
@@ -146,4 +146,3 @@
   </joint>
   </link>
-  </link>
 </robot>

Commit message: Add files via upload

File: src/my_robot/urdf/my_robot.xacro (robot description, xacro)
@@ -139,10 +139,40 @@
       </geometry>
     </visual>
-  <joint type="fixed" name="camer_joint">
+  <joint type="fixed" name="camera_joint">
     <origin xyz="0.2 0 0" rpy="0 0 0" />
-    <child link="left_wheel" />
+    <child link="camera" />
     <parent link="chassis" />
     <axis xyz="0 1 0" rpy="0 0 0" />
   </joint>
   </link>
+ <link name= 'hokuyo'/>
+  <pose>0 0 0 0 0 0</pose>
+   <inertial>
+      <mass value="1e-5" />
+      <origin xyz="0 0 0" rpy="0 0 0" />
+      <inertia
+        ixx="1e-6" ixy="0" ixz="0"
+        iyy="1e-6" iyz="0"
+        izz="1e-6"
+      />
+    </inertial>
+    <collision name='hokuyo_collision'>
+      <origin xyz="0 0 0" rpy=" 0 0 0"/>
+      <geometry>
+        <box size=".1 .1 .1"/>
+      </geometry>
+    </collision>
+ <visual name='hokuyo_visual'>
+      <origin xyz="0 0 0" rpy=" 0 0 0"/>
+      <geometry>
+        <box size=".1 .1 .1"/>
+      </geometry>
+    </visual>
+</link>
+  <joint type="fixed" name="hokuyo_joint">
+    <origin xyz="0.15 0 0.1" rpy="0 0 0" />
+    <child link="left_wheel" />
+    <parent link="hokuyo" />
+    <axis xyz="0 1 0" rpy="0 0 0" />
+  </joint>
 </robot>
